File: mcu.sch (KiCad schematic (older format))
At the start: 1 part

Commit message: Saving before reboot
Connections:
- net UART_TX: now reaches A?.1 (D1/TX)
- net UART_RX: now reaches A?.2 (D0/RX)
Changed lines of the file:
@@
 	1    0    0    -1
 $EndComp
+Text HLabel 4350 2700 0    50   Input ~ 0
+UART_RX
+Text HLabel 4350 2800 0    50   Input ~ 0
+UART_TX
+Wire Wire Line
+	4350 2700 4900 2700
+Wire Wire Line
+	4900 2800 4350 2800
 $EndSCHEMATC
