File: midi_io.sch (KiCad schematic (older format))
At the start: 0 parts

Commit message: Saving before reboot
Parts:
- added J? (x3): Conn_01x05_Male, symbol Connector:Conn_01x05_Male
Changed lines of the file:
@@
 $Descr A4 11693 8268
 encoding utf-8
-Sheet 1 5
+Sheet 4 5
 Title ""
 Date ""
@@
 Comment4 ""
 $EndDescr
+$Comp
+L Connector:Conn_01x05_Male J?
+U 1 1 5D75B250
+P 1750 1750
+F 0 "J?" H 1858 2131 50  0000 C CNN
+F 1 "Conn_01x05_Male" H 1858 2040 50  0000 C CNN
+F 2 "" H 1750 1750 50  0001 C CNN
+F 3 "~" H 1750 1750 50  0001 C CNN
+	1    1750 1750
+	1    0    0    -1
+$EndComp
+$Comp
+L Connector:Conn_01x05_Male J?
+U 1 1 5D75C545
+P 1750 2500
+F 0 "J?" H 1858 2881 50  0000 C CNN
+F 1 "Conn_01x05_Male" H 1858 2790 50  0000 C CNN
+F 2 "" H 1750 2500 50  0001 C CNN
+F 3 "~" H 1750 2500 50  0001 C CNN
+	1    1750 2500
+	1    0    0    -1
+$EndComp
+$Comp
+L Connector:Conn_01x05_Male J?
+U 1 1 5D75D52C
+P 5650 1700
+F 0 "J?" H 5622 1632 50  0000 R CNN
+F 1 "Conn_01x05_Male" H 5622 1723 50  0000 R CNN
+F 2 "" H 5650 1700 50  0001 C CNN
+F 3 "~" H 5650 1700 50  0001 C CNN
+	1    5650 1700
+	-1   0    0    1
+$EndComp
 $EndSCHEMATC
